File: QT-Wardriver-PCB/PCB/Wardriver-PCB.kicad_pcb (KiCad board)
At the start: 2 copper layers, 39 x 63 mm, 20 parts, among them J1 MICRO-SD CARD, J2 Conn_01x02_Female, J3 QWIIC, J3 Qwiic Connector, J5 Expansion Header, SW1 Up, SW2 Left, SW3 Right, SW4 Down, U1 XIAO ESP32-S2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

Commit message: changing board layout
Parts:
- added REF**: D_DO-41_SOD81_P7.62mm_Horizontal, Diode_THT:D_DO-41_SOD81_P7.62mm_Horizontal, F.Cu at (0.00, 9.50)
- added REF**: LiPo Backpack, Wardriver-Footprints:LiPo Backpack, B.Cu at (-17.8, 7.80)
- added REF**: SW_SPDT_PCM12, Button_Switch_SMD:SW_SPDT_PCM12, B.Cu at (17.8, 12.0)
- moved REF** 53.7 mm to (48.8, -14.2), turned to 0 degrees
- moved U1 30.1 mm to (0.00, 21.2), turned to 180 degrees
- moved J1 26.9 mm to (5.00, -9.45), turned to -90 degrees
- moved J2 20.4 mm to (-14.3, 0.41), turned to -90 degrees
- moved J5 15.4 mm to (13.5, 3.66), turned to 90 degrees
- moved J3 13.4 mm to (16.8, 21.9)
- moved J3 12.6 mm to (-16.8, 21.1)
- moved U2 2.21 mm to (-9.25, -11.8)
- moved SW1 0.88 mm to (0.00, 16.5)
- moved SW2 0.62 mm to (-7.25, 22.0)
- moved SW3 0.62 mm to (7.25, 22.0)
- moved SW4 0.38 mm to (0.00, 27.5)
Connections:
- J2 pad 1: +5V -> (no net)
- J2 pad 2: GND -> (no net)
- U3 pad 1: GND -> +3V3
- U3 pad 2: +3V3 -> GND
Routing:
- net +3V3: track 143.8 -> 0.00 mm, vias 2 -> 0
- net SCL: track 94.9 -> 0.00 mm, vias 2 -> 0
- net SDA: track 89.1 -> 0.00 mm, vias 1 -> 0
- net +5V: track 85.1 -> 0.00 mm, vias 3 -> 0
- net MOSI: track 51.7 -> 0.00 mm, vias 2 -> 0
- net MISO: track 50.9 -> 0.00 mm, vias 2 -> 0
- net SCK: track 47.8 -> 0.00 mm, vias 2 -> 0
- net LT-Btn: track 37.9 -> 0.00 mm, vias 1 -> 0
- net DN-Btn: track 30.4 -> 0.00 mm, vias 1 -> 0
- net UP-Btn: track 29.6 -> 0.00 mm, vias 1 -> 0
- net RT-Btn: track 24.3 -> 0.00 mm, vias 1 -> 0
- net TX: track 23.7 -> 0.00 mm
- net RX: track 23.5 -> 0.00 mm
- net GND: vias 7 -> 0
Other:
- board text removed: "DO NOT use USB & LiPo simultaneously w/out charging backpack!"

Commit message: publish v0.1 Cutie Wardriver design files
Parts:
- removed J5: Expansion Header, Connector_PinHeader_2.54mm:PinHeader_1x04_P2.54mm_Vertical_SMD_Pin1Right
- removed the REF** at (0.00, 9.50)
- removed the REF** at (-17.8, 7.80)
- removed the REF** at (48.8, -14.2)
- added G*** (x2): LOGO, LOGO, F.Cu at (-7.27, 27.9)
- added G***: LOGO, LOGO, B.Cu at (15.3, -21.9)
- added J6: Conn_01x05_Female, Connector_PinHeader_2.54mm:PinHeader_1x05_P2.54mm_Vertical_SMD_Pin1Left, B.Cu at (-4.75, -26.5)
- added U4: ~, PicoCharge:MiniMeter, B.Cu at (5.50, 15.5)
- J3: value QWIIC -> Qwiic Connector
- J4: renamed from U3; value ATGM336H -> SH1106
- SW5: renamed from REF**; value SW_SPDT_PCM12 -> SW_SPST
- moved SW5 35.5 mm to (-17.6, 9.50), turned to 90 degrees
- moved J2 33.6 mm to (7.50, 26.0), turned to 90 degrees
- moved U1 30.0 mm to (-9.19, -7.39), turned to 90 degrees
- moved U2 21.3 mm to (10.0, -2.75), turned to 0 degrees
- moved J3 0.88 mm to (16.8, 21.0)
- moved REF** 0.75 mm to (-5.00, -26.6)
- moved REF** 0.65 mm to (8.25, -27.3)
- moved J1 0.45 mm to (5.00, -9.00)
- moved J3 0.10 mm to (-16.8, 21.0)
Connections:
- J2 pad 1: (no net) -> VBAT
- J2 pad 2: (no net) -> GND
- J2 pad MP: (no net) -> GND
- J3 pad MP: (no net) -> GND (x2)
- REF** pad 2: (no net) -> GND
- SW5 pad 1: (no net) -> VBAT
- SW5 pad 2: (no net) -> Net-(SW5-B)
- U2 pad 5: (no net) -> unconnected-(U2-PPS-Pad5)
Routing:
- net SDA: track 0.00 -> 135.8 mm, vias 0 -> 3
- net +3V3: track 0.00 -> 135.8 mm, vias 0 -> 3
- net SCL: track 0.00 -> 115.7 mm, vias 0 -> 3
- net +5V: track 0.00 -> 83.4 mm
- net DN-Btn: track 0.00 -> 66.8 mm, vias 0 -> 1
- net VBAT: track 0.00 -> 64.1 mm
- net RT-Btn: track 0.00 -> 57.1 mm, vias 0 -> 1
- net LT-Btn: track 0.00 -> 49.3 mm, vias 0 -> 1
- net UP-Btn: track 0.00 -> 45.2 mm, vias 0 -> 1
- net TX: track 0.00 -> 32.4 mm
- net Net-(SW5-B): track 0.00 -> 28.0 mm
- net MISO: track 0.00 -> 26.9 mm, vias 0 -> 3
- net MOSI: track 0.00 -> 22.6 mm
- net SCK: track 0.00 -> 21.9 mm
- net RX: track 0.00 -> 13.3 mm
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Other:
- board text added: "Cutie"
- board text added: "Do not use LiPo without charge module."
- board text added: "Wardriver"
- board text removed: "Cut trace if using LiPo backpack."
- board text removed: "LiPo Battery"
- board text removed: "QT Wardriver"
