File: QT-Wardriver-PCB/PCB/Wardriver-PCB.kicad_sch (KiCad schematic)
At the start: 11 parts, among them J1 MICRO-SD CARD, J2 Conn_01x02_Female, J3 Qwiic Connector, J4 SH1106, J5 Expansion Header, SW1 Up, SW2 Left, SW3 Right, SW4 Down, U1 XIAO ESP32-S2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

Commit message: changing board layout
Parts:
- added D1: D_Small, symbol Device:D_Small
Connections:
- net +5V: now also D1.1 (K)
- net GND: now also J2.2 (Pin_2)
- net at J2.1 (Pin_1): now also D1.2 (A)
Changed lines of the file:
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@@
+    (stroke (width 0) (type default))
+  )
+  (wire (pts (xy 158.496 46.99) (xy 165.1 46.99))
     (stroke (width 0) (type default))
   )
@@
   )
   (wire (pts (xy 96.52 71.12) (xy 100.33 71.12))
+    (stroke (width 0) (type default))
+  )
+  (wire (pts (xy 158.369 44.45) (xy 160.02 44.45))
     (stroke (width 0) (type default))
   )
@@
     )
   )
+  (symbol (lib_id "power:GND") (at 158.496 46.99 0) (unit 1)
+    (in_bom yes) (on_board yes) (dnp no) (fields_autoplaced)
+    (property "Reference" "#PWR017" (at 158.496 53.34 0)
+      (effects (font (size 1.27 1.27)) hide)
+    )
+    (property "Value" "GND" (at 158.496 51.943 0)
+      (effects (font (size 1.27 1.27)))
+    )
+    (property "Footprint" "" (at 158.496 46.99 0)
+      (effects (font (size 1.27 1.27)) hide)
+    )
+    (property "Datasheet" "" (at 158.496 46.99 0)
+      (effects (font (size 1.27 1.27)) hide)
+    )
+    (pin "1")
+    (instances
+      (project "Wardriver-PCB"
+        (path "/b7a4ae1b-e08c-4382-98d6-abd93ff72581"
+          (reference "#PWR017") (unit 1)
+        )
+      )
+    )
+  )
   (symbol (lib_id "Switch:SW_Push") (at 142.24 60.96 0) (unit 1)
     (in_bom yes) (on_board yes) (dnp no)
@@
         (path "/e63e39d7-6ac0-4ffd-8aa3-1841a4541b55"
           (reference "J2") (unit 1)
+        )
+      )
+    )
+  )
+  (symbol (lib_id "Device:D_Small") (at 162.56 44.45 0) (unit 1)
+    (in_bom yes) (on_board yes) (dnp no)
+    (property "Reference" "D1" (at 162.814 38.608 0)
+      (effects (font (size 1.27 1.27)))
+    )
+    (property "Value" "D_Small" (at 165.354 40.767 0)
+      (effects (font (size 1.27 1.27)))
+    )
+    (property "Footprint" "" (at 162.56 44.45 90)
+      (effects (font (size 1.27 1.27)) hide)
+    )
+    (property "Datasheet" "~" (at 162.56 44.45 90)
+      (effects (font (size 1.27 1.27)) hide)
+    )
+    (pin "1")
+    (pin "2")
+    (instances
+      (project "Wardriver-PCB"
+        (path "/b7a4ae1b-e08c-4382-98d6-abd93ff72581"
+          (reference "D1") (unit 1)
         )
       )
@@
         )
       )
+    )
+  )
+  (symbol (lib_id "power:+5V") (at 158.369 44.45 0) (unit 1)
+    (in_bom yes) (on_board yes) (dnp no) (fields_autoplaced)
+    (property "Reference" "#PWR018" (at 158.369 48.26 0)
+      (effects (font (size 1.27 1.27)) hide)
+    )
+    (property "Value" "+5V" (at 158.369 39.37 0)
+      (effects (font (size 1.27 1.27)))
+    )
+    (property "Footprint" "" (at 158.369 44.45 0)
+      (effects (font (size 1.27 1.27)) hide)
+    )
+    (property "Datasheet" "" (at 158.369 44.45 0)
+      (effects (font (size 1.27 1.27)) hide)
+    )
+    (pin "1")
+    (instances
+      (project "Wardriver-PCB"
+        (path "/b7a4ae1b-e08c-4382-98d6-abd93ff72581"
+          (reference "#PWR018") (unit 1)
+        )
+      )

Commit message: publish v0.1 Cutie Wardriver design files
Parts:
- removed D1: D_Small, symbol Device:D_Small
- removed J5: Expansion Header, Connector_PinHeader_2.54mm:PinHeader_1x04_P2.54mm_Vertical_SMD_Pin1Right, symbol Connector:Conn_01x04_Female
- added J6: Conn_01x05_Female, Connector_PinHeader_2.54mm:PinHeader_1x05_P2.54mm_Vertical_SMD_Pin1Left, symbol Connector:Conn_01x05_Female
- added SW5: SW_SPST, symbol Switch:SW_SPST
- added U4: ~, PicoCharge:MiniMeter, symbol PicoCharge:MiniMeter
Connections:
- net +3V3: now also J6.3 (Pin_3)
- net +5V: now also J6.1 (Pin_1), U4.6 (VCC)
- net GND: now also J6.2 (Pin_2), U4.1 (GND), U4.5 (GND)
- net SCL: now also J6.5 (Pin_5), U4.4 (SCL)
- net SDA: now also J6.4 (Pin_4), U4.3 (SDA)
- net VBAT: now reaches J2.1 (Pin_1)
- net VBAT: now also SW5.1 (A), U4.7 (VBAT)
- new net: SW5.2 (B), U4.8 (EN)
Other:
- moved on the sheet: J2
