File: Cutie-Wardriver-PCB/PCB/Wardriver-PCB.kicad_pcb (KiCad board)
At the start: 2 copper layers, 39 x 63 mm, 24 parts, among them J1 MICRO-SD CARD, J2 Conn_01x02_Female, J3 Qwiic Connector, J4 SH1106, J6 Conn_01x05_Female, SW1 Up, SW2 Left, SW3 Right, SW4 Down, SW5 SW_SPST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

Commit message: push v0.2 files & image
Parts:
- added G***: LOGO, LOGO, F.Cu at (-23.9, 24.3)
- added G***: LOGO, LOGO, F.Cu at (-18.5, 13.1)
- added G***: LOGO, LOGO, F.Cu at (13.2, 14.4)
- added G***: LOGO, LOGO, F.Cu at (17.6, 18.0)
- added G***: LOGO, LOGO, F.Cu at (6.89, 26.5)
- added G***: LOGO, LOGO, F.Cu at (-15.2, 16.4)
- added G***: LOGO, LOGO, F.Cu at (18.6, 22.5)
- added G***: LOGO, LOGO, F.Cu at (-18.6, 20.4)
- added G***: LOGO, LOGO, F.Cu at (-12.6, 19.0)
- added G***: LOGO, LOGO, F.Cu at (8.61, 14.5)
- added G***: LOGO, LOGO, F.Cu at (-12.6, 24.9)
- added G***: LOGO, LOGO, F.Cu at (14.1, 23.7)
- added G***: LOGO, LOGO, F.Cu at (11.5, 27.7)
- added G***: LOGO, LOGO, F.Cu at (13.3, 17.9)
- added G***: LOGO, LOGO, F.Cu at (-9.09, 14.8)
- added G***: LOGO, LOGO, F.Cu at (-16.9, 24.2)
- moved U4 30.3 mm to (-5.76, -12.6), turned to -90 degrees
- moved SW5 24.5 mm to (-17.8, -15.0)
- moved U1 12.2 mm to (-9.20, 4.78)
- moved U2 9.92 mm to (9.49, 7.16), turned to 90 degrees
- moved J1 1.04 mm to (5.02, -10.0)
- moved G*** 0.54 mm to (15.4, -22.4)
- moved SW1 0.50 mm to (0.00, 16.0)
- moved SW2 0.50 mm to (-7.25, 21.5)
- moved SW3 0.50 mm to (7.25, 21.5)
- moved SW4 0.50 mm to (0.00, 27.0)
- moved J2 0.05 mm to (7.45, 26.0)
Connections:
- U4 pad 1: GND -> (no net)
Routing:
- net +5V: track 83.4 -> 55.4 mm
- net MOSI: track 22.6 -> 40.4 mm, vias 0 -> 2
- net Net-(SW5-B): track 28.0 -> 11.1 mm
- net LT-Btn: track 49.3 -> 33.0 mm
- net UP-Btn: track 45.2 -> 29.3 mm
- net SCK: track 21.9 -> 35.9 mm, vias 0 -> 2
- net MISO: track 26.9 -> 40.0 mm, vias 3 -> 2
- net RX: track 13.3 -> 24.6 mm
- net VBAT: track 64.1 -> 73.2 mm, vias 0 -> 3
- net TX: track 32.4 -> 24.0 mm
- net DN-Btn: track 66.8 -> 58.7 mm
- net RT-Btn: track 57.1 -> 61.8 mm
- net SDA: track 135.8 -> 139.4 mm, vias 3 -> 2
- net SCL: track 115.7 -> 114.5 mm, vias 3 -> 1
- net +3V3: track 135.8 -> 136.4 mm, vias 3 -> 2
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Other:
- board text added: "Do not attach LiPo without MiniMeter module."
- board text added: "ON"
- board text removed: "Do not use LiPo without charge module."
